Commit message: finish ICP

File: src/calibrator/urdf/ydlidar_eval.urdf (robot description, URDF)
Before this commit: robot ydlidarG4, 5 links, 4 joints
Joints:
- joint map2laser1: origin xyz=0 0 0 rpy=0 0 3.14 -> xyz=4 10 0 rpy=0 0 3.14
- joint map2laser2: origin xyz=0 0 0 rpy=0 0 3.14 -> xyz=0 10 0 rpy=0 0 3.14
- joint map2laser3: origin xyz=0 0 0 rpy=0 0 0 -> xyz=4 0 0 rpy=0 0 0

Commit message: finish calibration

File: src/calibrator/urdf/ydlidar_eval.urdf (robot description, URDF)
Before this commit: robot ydlidarG4, 5 links, 4 joints
Joints:
- joint map2laser1: origin xyz=4 10 0 rpy=0 0 3.14 -> xyz=4 0 0 rpy=0 0 3.14
- joint map2laser2: origin xyz=0 10 0 rpy=0 0 3.14 -> xyz=0 0 0 rpy=0 0 3.14
- joint map2laser3: origin xyz=4 0 0 rpy=0 0 0 -> xyz=4 -9 0 rpy=0 0 0
- joint map2laser4: origin xyz=0 0 0 rpy=0 0 0 -> xyz=0 -9 0 rpy=0 0 0
