Commit message: fix bug

File: src/calibrator/urdf/TG_new.urdf (robot description, URDF)
Before this commit: robot TG_ydlidar, 5 links, 4 joints
Joints:
- joint map2laser2: origin xyz=-2 5 0 rpy=0 0 0.785 -> xyz=-2 4 0 rpy=0 0 0.785
- joint map2laser4: origin xyz=2 5 0 rpy=0 0 0.785 -> xyz=2 4 0 rpy=0 0 0.785

Commit message: working on zero-meaned vector

File: src/calibrator/urdf/TG_new.urdf (robot description, URDF)
Before this commit: robot TG_ydlidar, 5 links, 4 joints
Joints:
- joint map2laser3: origin xyz=-2 -5 0 rpy=0 0 -1.57 -> xyz=-2 -5 0 rpy=0 0 3.14

Commit message: add GoalPose topic

File: src/calibrator/urdf/TG_new.urdf (robot description, URDF)
Before this commit: robot TG_ydlidar, 5 links, 4 joints
Joints:
- joint map2laser3: origin xyz=-2 -5 0 rpy=0 0 3.14 -> xyz=-2 -5 0 rpy=0 0 -1.57
- joint map2laser4: origin xyz=2 4 0 rpy=0 0 0.785 -> xyz=2 3 0 rpy=0 0 0.785

Commit message: modify urdf

File: src/calibrator/urdf/TG_new.urdf (robot description, URDF)
Before this commit: robot TG_ydlidar, 5 links, 4 joints
Joints:
- joint map2laser3: origin xyz=-2 -5 0 rpy=0 0 -1.57 -> xyz=-2 -5 0 rpy=0 0 0.785
